File: Test2_Github.kicad_pcb (KiCad board)
At the start: 2 copper layers, 37.1 x 37.1 mm, 7 parts, among them SW2 SW_MEC_5E

Commit message: Routing done
Parts:
- moved R2 7.95 mm to (96.4, 64.5), turned to 180 degrees
Connections:
- D2 pad 1: Net-(D1-K) -> Net-(D2-K)
- D2 pad 2: Net-(D2-A) -> Net-(D1-A)
- R1 pad 1: Net-(D1-A) -> Net-(D1-K)
- R2 pad 1: Net-(D2-A) -> Net-(D2-K)
Routing:
- net Net-(BT1-+): track 0.00 -> 51.8 mm
- net Net-(D1-A): track 0.00 -> 48.0 mm
- net Net-(BT1--): track 0.00 -> 34.2 mm
- net Net-(D1-K): track 0.00 -> 11.5 mm
- net Net-(D2-K): track 0.00 -> 8.25 mm
Changed lines of the file:
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@@
   (net 3 "Net-(D1-K)")
   (net 4 "Net-(D1-A)")
-  (net 5 "Net-(D2-A)")
+  (net 5 "Net-(D2-K)")
   (footprint "Resistor_THT:R_Axial_DIN0204_L3.6mm_D1.6mm_P7.62mm_Horizontal" (layer "F.Cu")
-    (at 88.4936 64.4906)
+    (at 96.4438 64.4652 180)
     (descr "Resistor, Axial_DIN0204 series, Axial, Horizontal, pin pitch=7.62mm, 0.167W, length*diameter=3.6*1.6mm^2, http://cdn-reichelt.de/documents/datenblatt/B400/1_4W%23YAG.pdf")
     (tags "Resistor Axial_DIN0204 series Axial Horizontal pin pitch 7.62mm 0.167W length 3.6mm diameter 1.6mm")
@@
     (fp_line (start 7.62 0) (end 5.61 0)
       (stroke (width 0.1) (type solid)) (layer "F.Fab"))
-    (pad "1" thru_hole circle (at 0 0) (size 1.4 1.4) (drill 0.7) (layers "*.Cu" "*.Mask")
-      (net 5 "Net-(D2-A)") (pintype "passive"))
-    (pad "2" thru_hole oval (at 7.62 0) (size 1.4 1.4) (drill 0.7) (layers "*.Cu" "*.Mask")
+    (pad "1" thru_hole circle (at 0 0 180) (size 1.4 1.4) (drill 0.7) (layers "*.Cu" "*.Mask")
+      (net 5 "Net-(D2-K)") (pintype "passive"))
+    (pad "2" thru_hole oval (at 7.62 0 180) (size 1.4 1.4) (drill 0.7) (layers "*.Cu" "*.Mask")
       (net 2 "Net-(BT1--)") (pintype "passive"))
     (model "${KICAD6_3DMODEL_DIR}/Resistor_THT.3dshapes/R_Axial_DIN0204_L3.6mm_D1.6mm_P7.62mm_Horizontal.wrl"
@@
       (stroke (width 0.1) (type solid)) (fill none) (layer "F.Fab"))
     (pad "1" thru_hole rect (at 0 0) (size 1.8 1.8) (drill 0.9) (layers "*.Cu" "*.Mask")
-      (net 3 "Net-(D1-K)") (pinfunction "K") (pintype "passive"))
+      (net 5 "Net-(D2-K)") (pinfunction "K") (pintype "passive"))
     (pad "2" thru_hole circle (at 2.54 0) (size 1.8 1.8) (drill 0.9) (layers "*.Cu" "*.Mask")
-      (net 5 "Net-(D2-A)") (pinfunction "A") (pintype "passive"))
+      (net 4 "Net-(D1-A)") (pinfunction "A") (pintype "passive"))
     (model "${KICAD6_3DMODEL_DIR}/LED_THT.3dshapes/LED_D5.0mm_Clear.wrl"
       (offset (xyz 0 0 0))
@@
       (stroke (width 0.1) (type solid)) (layer "F.Fab"))
     (pad "1" thru_hole circle (at 0 0) (size 1.4 1.4) (drill 0.7) (layers "*.Cu" "*.Mask")
-      (net 4 "Net-(D1-A)") (pintype "passive"))
+      (net 3 "Net-(D1-K)") (pintype "passive"))
     (pad "2" thru_hole oval (at 7.62 0) (size 1.4 1.4) (drill 0.7) (layers "*.Cu" "*.Mask")
       (net 2 "Net-(BT1--)") (pintype "passive"))
@@
   (gr_circle (center 92.2528 61.7728) (end 103.9114 76.1746)
     (stroke (width 0.1) (type default)) (fill none) (layer "Edge.Cuts"))
+  (segment (start 89.2834 70.5358) (end 95.7834 70.5358) (width 0.25) (layer "F.Cu") (net 1))
+  (segment (start 85.7274 52.7812) (end 85.7274 54.968) (width 0.25) (layer "F.Cu") (net 1))
+  (segment (start 87.5284 63.4238) (end 88.9254 63.4238) (width 0.25) (layer "F.Cu") (net 1))
+  (segment (start 87.1474 56.388) (end 91.8488 56.388) (width 0.25) (layer "F.Cu") (net 1))
+  (segment (start 89.2834 70.5358) (end 87.5284 68.7808) (width 0.25) (layer "F.Cu") (net 1))
+  (segment (start 85.7274 54.968) (end 87.1474 56.388) (width 0.25) (layer "F.Cu") (net 1))
+  (segment (start 91.8488 56.388) (end 95.354 52.8828) (width 0.25) (layer "F.Cu") (net 1))
+  (segment (start 95.354 56.9952) (end 95.354 52.8828) (width 0.25) (layer "F.Cu") (net 1))
+  (segment (start 89.2834 75.0358) (end 89.2834 70.5358) (width 0.25) (layer "F.Cu") (net 1))
+  (segment (start 95.7834 75.0358) (end 95.7834 70.5358) (width 0.25) (layer "F.Cu") (net 1))
+  (segment (start 87.5284 68.7808) (end 87.5284 63.4238) (width 0.25) (layer "F.Cu") (net 1))
+  (segment (start 88.9254 63.4238) (end 95.354 56.9952) (width 0.25) (layer "F.Cu") (net 1))
+  (segment (start 96.1898 61.6712) (end 99.314 58.547) (width 0.25) (layer "F.Cu") (net 2))
+  (segment (start 94.9198 62.9412) (end 96.1898 61.6712) (width 0.25) (layer "F.Cu") (net 2))
+  (segment (start 88.8238 64.4652) (end 90.3478 62.9412) (width 0.25) (layer "F.Cu") (net 2))
+  (segment (start 96.8248 48.641) (end 99.314 51.1302) (width 0.25) (layer "F.Cu") (net 2))
+  (segment (start 89.6874 50.3174) (end 91.3638 48.641) (width 0.25) (layer "F.Cu") (net 2))
+  (segment (start 91.3638 48.641) (end 96.8248 48.641) (width 0.25) (layer "F.Cu") (net 2))
+  (segment (start 99.314 51.1302) (end 99.314 52.8828) (width 0.25) (layer "F.Cu") (net 2))
+  (segment (start 89.6874 52.7812) (end 89.6874 50.3174) (width 0.25) (layer "F.Cu") (net 2))
+  (segment (start 99.314 58.547) (end 99.314 52.8828) (width 0.25) (layer "F.Cu") (net 2))
+  (segment (start 90.3478 62.9412) (end 94.9198 62.9412) (width 0.25) (layer "F.Cu") (net 2))
+  (segment (start 87.8698 60.9712) (end 79.567 60.9712) (width 0.25) (layer "F.Cu") (net 3))
+  (segment (start 79.567 60.9712) (end 78.0034 62.5348) (width 0.25) (layer "F.Cu") (net 3))
+  (segment (start 88.5698 61.6712) (end 87.8698 60.9712) (width 0.25) (layer "F.Cu") (net 3))
+  (segment (start 80.5434 62.5348) (end 84.2772 66.2686) (width 0.25) (layer "F.Cu") (net 4))
+  (segment (start 96.9772 78.486) (end 102.5144 72.9488) (width 0.25) (layer "F.Cu") (net 4))
+  (segment (start 102.5144 72.7456) (end 106.7512 68.5088) (width 0.25) (layer "F.Cu") (net 4))
+  (segment (start 86.6902 78.486) (end 96.9772 78.486) (width 0.25) (layer "F.Cu") (net 4))
+  (segment (start 106.7512 68.5088) (end 106.7512 63.2968) (width 0.25) (layer "F.Cu") (net 4))
+  (segment (start 102.5144 72.9488) (end 102.5144 72.7456) (width 0.25) (layer "F.Cu") (net 4))
+  (segment (start 84.2772 66.2686) (end 84.2772 76.073) (width 0.25) (layer "F.Cu") (net 4))
+  (segment (start 84.2772 76.073) (end 86.6902 78.486) (width 0.25) (layer "F.Cu") (net 4))
+  (segment (start 96.4438 64.4652) (end 97.6122 63.2968) (width 0.25) (layer "F.Cu") (net 5))
+  (segment (start 97.6122 63.2968) (end 104.2112 63.2968) (width 0.25) (layer "F.Cu") (net 5))
 )
